File: aquos_pcb/aquos_pcb.kicad_pcb (KiCad board)
At the start: 2 copper layers, 23 parts, among them J1 Conn_01x04, J2 Conn_01x04, J3 Conn_01x04, J4 Conn_01x04, J5 Conn_01x02, SW1 SW_SPDT, U1 ESP32-DEVKIT-V1, U2 TXE0108E, U3 TP4056_MICRO-USB_CHARGER_-_1A

Commit message: ready to print
Parts:
- removed C1: C_Polarized, Capacitor_THT:CP_Radial_D6.3mm_P2.50mm
- added R13: 1k5, Resistor_THT:R_Axial_DIN0204_L3.6mm_D1.6mm_P5.08mm_Horizontal, F.Cu at (104.5, 128.0)
- added R14: 3k3, Resistor_THT:R_Axial_DIN0204_L3.6mm_D1.6mm_P5.08mm_Horizontal, F.Cu at (99.2, 128.0)
- R11: value 1k8 -> 3k3
- R12: value 1k8 -> 330
- R5, R6, R7: value 1k8 -> 1k5
- U3: value TP4056_MICRO-USB_CHARGER_-_1A -> ~; footprint TP4056_MICRO-USB_CHARGER_-_1A:MODULE_TP4056_MICRO-USB_CHARGER_-_1A -> USB-MICRO-B-MODULE:USB-MICRO-B-MODULE
- moved J5 97.2 mm to (184.5, 74.2), turned to 180 degrees
- moved SW1 33.8 mm to (170.5, 51.5), turned to 180 degrees
- moved D1 9.49 mm to (165.8, 65.5)
- moved R12 7.19 mm to (177.0, 73.8)
- moved U3 6.29 mm to (190.7, 54.0), turned to 0 degrees
- moved U2 0.68 mm to (166.8, 97.4), turned to 180 degrees
Connections:
- J1 pad 2: GND -> GND2
- J2 pad 2: GND -> GND2
- J3 pad 2: GND -> GND2
- J4 pad 1: +3.3V -> Net-(J4-Pin_1)
- J4 pad 4: GND -> GND2
- R10 pad 1: GND -> GND2
- R8 pad 1: GND -> GND2
- R9 pad 1: GND -> GND2
- U1 pad 29: GND -> GND2
- U2 pad 12: Net-(DS1-RS) -> Net-(DS1-D7)
- U2 pad 13: Net-(DS1-E) -> Net-(DS1-D6)
- U2 pad 14: unconnected-(U2-B3-Pad14) -> Net-(DS1-D5)
- U2 pad 16: Net-(DS1-D5) -> Net-(DS1-E)
- U2 pad 17: Net-(DS1-D6) -> Net-(DS1-RS)
- U2 pad 18: Net-(DS1-D7) -> unconnected-(U2-B7-Pad18)
- U2 pad 2: /RS -> /D7
- U2 pad 3: /EN -> /D6
- U2 pad 4: unconnected-(U2-A3-Pad4) -> /D5
- U2 pad 6: /D5 -> /EN
- U2 pad 7: /D6 -> /RS
- U2 pad 8: /D7 -> unconnected-(U2-A7-Pad8)
Routing:
- net GND: track 584.5 -> 327.1 mm
- net GND2: track 0.00 -> 233.5 mm
- net +3.3V: track 116.3 -> 43.5 mm
- net Net-(J4-Pin_1): track 0.00 -> 34.9 mm
- net Net-(SW1-B): track 11.1 -> 27.4 mm
- net VCC: track 449.8 -> 463.5 mm
- net Net-(DS1-VO): track 94.9 -> 101.9 mm
- net Net-(DS1-RS): track 25.0 -> 31.4 mm
- net Net-(DS1-E): track 23.0 -> 29.2 mm
- net /D7: track 42.6 -> 37.0 mm
- net /D6: track 39.0 -> 33.5 mm
- net Net-(DS1-D7): track 14.2 -> 19.1 mm
- net Net-(DS1-D6): track 14.5 -> 19.1 mm
- net Net-(DS1-D5): track 14.8 -> 19.1 mm
- net Net-(DS1-D4): track 15.0 -> 19.1 mm
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