File: aquos_pcb/aquos_pcb.kicad_sch (KiCad schematic)
At the start: 21 parts, among them J1 Conn_01x04, J2 Conn_01x04, J3 Conn_01x04, J4 Conn_01x04, J5 Conn_01x02, SW1 SW_SPDT, U1 ESP32-DEVKIT-V1, U2 TXE0108E, U3 TP4056_MICRO-USB_CHARGER_-_1A

Commit message: ready to print
Parts:
- removed C1: C_Polarized, Capacitor_THT:CP_Radial_D6.3mm_P2.50mm, symbol Device:C_Polarized
- removed U3: TP4056_MICRO-USB_CHARGER_-_1A, TP4056_MICRO-USB_CHARGER_-_1A:MODULE_TP4056_MICRO-USB_CHARGER_-_1A, symbol TP4056_MICRO-USB_CHARGER_-_1A:TP4056_MICRO-USB_CHARGER_-_1A
- added R13: 1k5, Resistor_THT:R_Axial_DIN0204_L3.6mm_D1.6mm_P5.08mm_Horizontal, symbol Device:R
- added R14: 3k3, Resistor_THT:R_Axial_DIN0204_L3.6mm_D1.6mm_P5.08mm_Horizontal, symbol Device:R
- added U3: (no value), USB-MICRO-B-MODULE:USB-MICRO-B-MODULE, symbol USB_MICRO_B_MODULE:USB-MICRO-B-MODULE
- R11: value 1k8 -> 3k3
- R12: value 1k8 -> 330
- R5, R6, R7: value 1k8 -> 1k5
Connections:
- net +3.3V: no longer J4.1 (Pin_1)
- net D5: now also U2.4 (A3); no longer U2.6 (A5)
- net D6: now also U2.3 (A2); no longer U2.7 (A6)
- net D7: now also U2.2 (A1); no longer U2.8 (A7)
- net EN: now also U2.6 (A5); no longer U2.3 (A2)
- net GND: now also U3.1 (GND); no longer J1.2 (Pin_2), J2.2 (Pin_2), J3.2 (Pin_2), J4.4 (Pin_4), R10.1, R8.1, R9.1, U1.29 (GND)
- net RS: now also U2.7 (A6); no longer U2.2 (A1)
- net VCC: now also R13.2
- net at U2.12 (B1): now also DS1.14 (D7); no longer DS1.4 (RS)
- net at U2.13 (B2): now also DS1.13 (D6); no longer DS1.6 (E)
- net at U2.14 (B3): now also DS1.12 (D5)
- net at U2.16 (B5): now also DS1.6 (E); no longer DS1.12 (D5)
- net at U2.17 (B6): now also DS1.4 (RS); no longer DS1.13 (D6)
- net at U2.18 (B7): no longer DS1.14 (D7)
- net at SW1.2 (B): now also U3.5 (VBUS)
- new net: J4.1 (Pin_1), R13.1, R14.2
- new net GND2: J1.2 (Pin_2), J2.2 (Pin_2), J3.2 (Pin_2), J4.4 (Pin_4), R10.1, R14.1, R8.1, R9.1, U1.29 (GND)
